File: PCB/Gantry_PCBv2/Gantry_PCBv2.kicad_sch (KiCad schematic)
At the start: 64 parts, among them J1 Conn_01x14, J10 B2B-XH-A_LF__SN_, J11 B2B-XH-A_LF__SN_, J12 B2B-XH-A_LF__SN_, J13 Conn_01x03_Pin, J17 B2B-XH-A_LF__SN_, J2 Conn_01x14, J20 TYPE-C-31-M-12, J3 Conn_01x10, J4 Screw_Terminal_01x02, J5 DCJ200-10-A-XX-X_REVA, J6 Conn_01x04_Pin, J7 Conn_01x04_Pin, J8 Conn_01x04_Pin, J9 Conn_01x04_Pin, Q1 SS8050, Q2 SS8050, SW7 SW_0, SW8 SW_EN, U1 ESP32-WROOM-32E, U2 CH340C, U3 TB6612FNG H-bridge Motor Driv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, U4 LM2576S-5, U5 AMS1117-3.3, U6 DRV8825_STEPPER_MOTOR_DRIVER_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, U7 DRV8825_STEPPER_MOTOR_DRIVER_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, U8 DRV8825_STEPPER_MOTOR_DRIVER_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, U9 DRV8825_STEPPER_MOTOR_DRIVER_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

Commit message: Component Placement done
Parts:
- J10, J11, J12, J17: footprint JST Connector:2 Pin JST Connector -> 2 Pin JST_Power&Motors:JST_B2B-XH-A_LF__SN_
- U1: footprint ESP-32:ESP32-WROOM-32E__4MB_HIGH_TEMP_ -> ESP32-WROOM:XCVR_ESP32-WROOM-32E__4MB_HIGH_TEMP_
- U3: footprint Motor Drivers:TB6612FNG -> motor_driver:TB6612FNG
- U6, U7, U8, U9: footprint DRV8825_STEPPER_MOTOR_DRIVER_CARRIER:IC_DRV8825_STEPPER_MOTOR_DRIVER_CARRIER -> DRV8825_STEPPER_MOTOR_DRIVER_CARRIER (1):IC_DRV8825_STEPPER_MOTOR_DRIVER_CARRIER
Changed lines of the file:
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@@
 			)
 		)
-		(property "Footprint" "ESP-32:ESP32-WROOM-32E__4MB_HIGH_TEMP_"
+		(property "Footprint" "ESP32-WROOM:XCVR_ESP32-WROOM-32E__4MB_HIGH_TEMP_"
 			(at 54.1274 103.9876 0)
 			(effects
@@
 			)
 		)
-		(property "Footprint" "DRV8825_STEPPER_MOTOR_DRIVER_CARRIER:IC_DRV8825_STEPPER_MOTOR_DRIVER_CARRIER"
+		(property "Footprint" "DRV8825_STEPPER_MOTOR_DRIVER_CARRIER (1):IC_DRV8825_STEPPER_MOTOR_DRIVER_CARRIER"
 			(at 186.69 151.13 0)
 			(effects
@@
 			)
 		)
-		(property "Footprint" "Motor Drivers:TB6612FNG"
+		(property "Footprint" "motor_driver:TB6612FNG"
 			(at 256.4892 47.8028 0)
 			(effects
@@
 			)
 		)
-		(property "Footprint" "JST Connector:2 Pin JST Connector"
+		(property "Footprint" "2 Pin JST_Power&Motors:JST_B2B-XH-A_LF__SN_"
 			(at 171.45 199.39 0)
 			(effects
@@
 			)
 		)
-		(property "Footprint" "DRV8825_STEPPER_MOTOR_DRIVER_CARRIER:IC_DRV8825_STEPPER_MOTOR_DRIVER_CARRIER"
+		(property "Footprint" "DRV8825_STEPPER_MOTOR_DRIVER_CARRIER (1):IC_DRV8825_STEPPER_MOTOR_DRIVER_CARRIER"
 			(at 186.69 105.41 0)
 			(effects
@@
 			)
 		)
-		(property "Footprint" "JST Connector:2 Pin JST Connector"
+		(property "Footprint" "2 Pin JST_Power&Motors:JST_B2B-XH-A_LF__SN_"
 			(at 125.73 198.12 0)
 			(effects
@@
 			)
 		)
-		(property "Footprint" "JST Connector:2 Pin JST Connector"
+		(property "Footprint" "2 Pin JST_Power&Motors:JST_B2B-XH-A_LF__SN_"
 			(at 125.73 210.82 0)
 			(effects
@@
 			)
 		)
-		(property "Footprint" "DRV8825_STEPPER_MOTOR_DRIVER_CARRIER:IC_DRV8825_STEPPER_MOTOR_DRIVER_CARRIER"
+		(property "Footprint" "DRV8825_STEPPER_MOTOR_DRIVER_CARRIER (1):IC_DRV8825_STEPPER_MOTOR_DRIVER_CARRIER"
 			(at 245.11 106.68 0)
 			(effects
@@
 			)
 		)
-		(property "Footprint" "JST Connector:2 Pin JST Connector"
+		(property "Footprint" "2 Pin JST_Power&Motors:JST_B2B-XH-A_LF__SN_"
 			(at 125.73 186.69 0)
 			(effects
@@
 			)
 		)
-		(property "Footprint" "DRV8825_STEPPER_MOTOR_DRIVER_CARRIER:IC_DRV8825_STEPPER_MOTOR_DRIVER_CARRIER"
+		(property "Footprint" "DRV8825_STEPPER_MOTOR_DRIVER_CARRIER (1):IC_DRV8825_STEPPER_MOTOR_DRIVER_CARRIER"
 			(at 245.11 149.86 0)
 			(effects
